File: kicad/sensorboard.kicad_sch (KiCad schematic)
At the start: 2 parts, among them U3 TMP117MAIDRVT, U5 SHT40-AD1B-R2

Commit message: Updated USB module
Other:
- company: (none) -> University of Oulu
Changed lines of the file:
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@@
 (kicad_sch (version 20230121) (generator eeschema)
   (paper "A4")
+  (title_block
+    (company "University of Oulu")
+  )
   (symbol (lib_id "SHT40-AD1B-R2:SHT40-AD1B-R2") (at 120.65 101.6 0) (unit 1)
     (in_bom yes) (on_board yes) (dnp no) (fields_autoplaced)
