File: kicad/voltage_regulator.kicad_sch (KiCad schematic)
At the start: 3 parts, among them U6 TCR2EF33

Commit message: Updated nrf9160 symbols for easier use, added sim card holder and doc, added first connections to mcu
Parts:
- renumbered C1 to C20, C2 to C21
Changed lines of the file:
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@@
   (symbol (lib_id "Device:C") (at 88.9 82.55 0) (unit 1)
     (in_bom yes) (on_board yes) (dnp no) (fields_autoplaced)
-    (property "Reference" "C1" (at 92.71 81.915 0)
+    (property "Reference" "C20" (at 92.71 81.915 0)
       (effects (font (size 1.27 1.27)) (justify left))
     )
@@
       (project "IoT_sulari"
         (path "/184b47ed-2c2b-4c02-be35-d18f4f4e5685/900a775e-83e7-4530-ab2f-7e5f26c05ece"
-          (reference "C1") (unit 1)
+          (reference "C20") (unit 1)
         )
       )
@@
   (symbol (lib_id "Device:C") (at 165.1 83.82 0) (unit 1)
     (in_bom yes) (on_board yes) (dnp no) (fields_autoplaced)
-    (property "Reference" "C2" (at 168.91 83.185 0)
+    (property "Reference" "C21" (at 168.91 83.185 0)
       (effects (font (size 1.27 1.27)) (justify left))
     )
@@
       (project "IoT_sulari"
         (path "/184b47ed-2c2b-4c02-be35-d18f4f4e5685/900a775e-83e7-4530-ab2f-7e5f26c05ece"
-          (reference "C2") (unit 1)
+          (reference "C21") (unit 1)
         )
       )

Commit message: added power jack and usb connector
Parts:
- added J2: 694106106102, CONN4_8106102_WRE, symbol 694106106102:694106106102
Connections:
- net GND: now also J2.2
- net VBUS: no longer names the net of C20.1, U6.1 (VIN)
- net VBUS: now also J2.1, J2.4 (1)
Other:
- note added: "Connect usb ground to pin 3?"
Changed lines of the file:
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@@
 (kicad_sch (version 20230121) (generator eeschema)
   (paper "A4")
+  (junction (at 69.85 69.85) (diameter 0) (color 0 0 0 0)
+  )
   (junction (at 165.1 78.74) (diameter 0) (color 0 0 0 0)
   )
   (junction (at 99.06 78.74) (diameter 0) (color 0 0 0 0)
   )
+  (junction (at 88.9 92.71) (diameter 0) (color 0 0 0 0)
+  )
   (junction (at 99.06 92.71) (diameter 0) (color 0 0 0 0)
   )
@@
     (stroke (width 0) (type default))
   )
+  (wire (pts (xy 69.85 69.85) (xy 69.85 68.58))
+    (stroke (width 0) (type default))
+  )
   (wire (pts (xy 99.06 78.74) (xy 102.87 78.74))
     (stroke (width 0) (type default))
   )
+  (wire (pts (xy 68.58 81.28) (xy 77.47 81.28))
+    (stroke (width 0) (type default))
+  )
   (wire (pts (xy 148.59 78.74) (xy 165.1 78.74))
     (stroke (width 0) (type default))
   )
+  (wire (pts (xy 69.85 71.12) (xy 69.85 69.85))
+    (stroke (width 0) (type default))
+  )
   (wire (pts (xy 165.1 78.74) (xy 165.1 80.01))
     (stroke (width 0) (type default))
@@
     (stroke (width 0) (type default))
   )
-  (wire (pts (xy 92.71 69.85) (xy 99.06 69.85))
+  (wire (pts (xy 68.58 71.12) (xy 69.85 71.12))
+    (stroke (width 0) (type default))
+  )
+  (wire (pts (xy 69.85 69.85) (xy 99.06 69.85))
     (stroke (width 0) (type default))
   )
@@
     (stroke (width 0) (type default))
   )
+  (wire (pts (xy 77.47 92.71) (xy 88.9 92.71))
+    (stroke (width 0) (type default))
+  )
+  (wire (pts (xy 77.47 81.28) (xy 77.47 92.71))
+    (stroke (width 0) (type default))
+  )
   (wire (pts (xy 88.9 86.36) (xy 88.9 92.71))
     (stroke (width 0) (type default))
@@
     (stroke (width 0) (type default))
   )
-  (text "Place battery bank connector here" (at 81.28 69.85 0)
+  (wire (pts (xy 68.58 68.58) (xy 69.85 68.58))
+    (stroke (width 0) (type default))
+  )
+  (text "Connect usb ground to pin 3?" (at 67.31 74.93 0)
+    (effects (font (size 1.27 1.27)) (justify left bottom))
+  )
+  (text "Place battery bank connector here" (at 95.25 57.15 0)
     (effects (font (size 1.27 1.27)) (justify right bottom))
-  )
-  (global_label "VBUS" (shape input) (at 92.71 69.85 180) (fields_autoplaced)
-    (effects (font (size 1.27 1.27)) (justify right))
-    (property "Intersheetrefs" "${INTERSHEET_REFS}" (at 84.9056 69.85 0)
-      (effects (font (size 1.27 1.27)) (justify right) hide)
-    )
   )
   (global_label "V_R_ctrl" (shape input) (at 151.13 83.82 0) (fields_autoplaced)
@@
         )
       )
+    )
+  )
+  (symbol (lib_id "694106106102:694106106102") (at 68.58 68.58 0) (mirror y) (unit 1)
+    (in_bom yes) (on_board yes) (dnp no)
+    (property "Reference" "J2" (at 39.37 73.66 0)
+      (effects (font (size 1.524 1.524)) (justify left))
+    )
+    (property "Value" "694106106102" (at 39.37 76.2 0)
+      (effects (font (size 1.524 1.524)) (justify left))
+    )
+    (property "Footprint" "CONN4_8106102_WRE" (at 58.42 65.024 0)
+      (effects (font (size 1.524 1.524)) hide)
+    )
+    (property "Datasheet" "" (at 68.58 68.58 0)
+      (effects (font (size 1.524 1.524)))
+    )
+    (pin "1")
+    (pin "2")
+    (pin "3")
+    (pin "4")
+    (instances
+      (project "IoT_sulari"
+        (path "/184b47ed-2c2b-4c02-be35-d18f4f4e5685/900a775e-83e7-4530-ab2f-7e5f26c05ece"
+          (reference "J2") (unit 1)
+        )
+      )

Commit message: Updated USB module
Other:
- company: (none) -> University of Oulu
Changed lines of the file:
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@@
 (kicad_sch (version 20230121) (generator eeschema)
   (paper "A4")
+  (title_block
+    (company "University of Oulu")
+  )
   (junction (at 69.85 69.85) (diameter 0) (color 0 0 0 0)
   )
