File: kicad/voltage_regulator.kicad_sch (KiCad schematic)
At the start: 5 parts, among them J20 694106106102, U20 MIC5219-3.3YM5-TR

Commit message: Updated PCB design rules and layout to correct placing around nRF9160
Changed lines of the file:
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@@
   )
   (symbol (lib_id "Device:C") (at 69.85 71.12 0) (unit 1)
-    (in_bom yes) (on_board yes) (dnp no) (fields_autoplaced)
-    (property "Reference" "C20" (at 73.66 70.485 0)
+    (in_bom yes) (on_board yes) (dnp no)
+    (property "Reference" "C20" (at 64.77 68.58 0)
       (effects (font (size 1.27 1.27)) (justify left))
     )
-    (property "Value" "100n" (at 73.66 73.025 0)
+    (property "Value" "100n" (at 64.135 73.66 0)
       (effects (font (size 1.27 1.27)) (justify left))
     )

Commit message: routing
Changed lines of the file:
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@@
     (stroke (width 0) (type default))
   )
-  (wire (pts (xy 156.21 53.34) (xy 156.21 64.77))
+  (wire (pts (xy 156.21 59.055) (xy 156.21 64.77))
     (stroke (width 0) (type default))
   )
@@
     )
   )
-  (symbol (lib_id "power:+3.3V") (at 156.21 53.34 0) (unit 1)
+  (symbol (lib_id "power:+3.3V") (at 156.21 59.055 0) (unit 1)
     (in_bom yes) (on_board yes) (dnp no) (fields_autoplaced)
-    (property "Reference" "#PWR01" (at 156.21 57.15 0)
+    (property "Reference" "#PWR01" (at 156.21 62.865 0)
       (effects (font (size 1.27 1.27)) hide)
     )
-    (property "Value" "+3.3V" (at 156.21 49.53 0)
+    (property "Value" "+3.3V" (at 156.21 55.245 0)
       (effects (font (size 1.27 1.27)))
     )
-    (property "Footprint" "" (at 156.21 53.34 0)
+    (property "Footprint" "" (at 156.21 59.055 0)
       (effects (font (size 1.27 1.27)) hide)
     )
-    (property "Datasheet" "" (at 156.21 53.34 0)
+    (property "Datasheet" "" (at 156.21 59.055 0)
       (effects (font (size 1.27 1.27)) hide)
     )

Commit message: Finished routing and added vias
Changed lines of the file:
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@@
     (effects (font (size 1.27 1.27)) (justify left bottom))
+  )
+  (global_label "+3.3V" (shape input) (at 156.21 59.055 90) (fields_autoplaced)
+    (effects (font (size 1.27 1.27)) (justify left))
+    (property "Intersheetrefs" "${INTERSHEET_REFS}" (at 156.21 50.4644 90)
+      (effects (font (size 1.27 1.27)) (justify left) hide)
+    )
   )
   (symbol (lib_id "Device:C") (at 142.24 76.2 0) (unit 1)
@@
         )
       )
-    )
-  )
-  (symbol (lib_id "power:+3.3V") (at 156.21 59.055 0) (unit 1)
-    (in_bom yes) (on_board yes) (dnp no) (fields_autoplaced)
-    (property "Reference" "#PWR01" (at 156.21 62.865 0)
-      (effects (font (size 1.27 1.27)) hide)
-    )
-    (property "Value" "+3.3V" (at 156.21 55.245 0)
-      (effects (font (size 1.27 1.27)))
-    )
-    (property "Footprint" "" (at 156.21 59.055 0)
-      (effects (font (size 1.27 1.27)) hide)
-    )
-    (property "Datasheet" "" (at 156.21 59.055 0)
-      (effects (font (size 1.27 1.27)) hide)
-    )
-    (pin "1")
-    (instances
-      (project "IoT_sulari"
-        (path "/184b47ed-2c2b-4c02-be35-d18f4f4e5685/900a775e-83e7-4530-ab2f-7e5f26c05ece"
-          (reference "#PWR01") (unit 1)
-        )
-      )
