File: kicad/IoT_sulari_sensorboard/IoT_sulari_sensorboard.kicad_pcb (KiCad board)
At the start: 2 copper layers, 8 parts, among them J1 20021121-00010C4LF, U1 SHT40-AD1B-R3, U2 TMP117MAIDRVT

Commit message: sensorboard pcb drawing
Parts:
- moved C1 24.3 mm to (135.0, 94.0), turned to 180 degrees
- moved C2 18.9 mm to (141.1, 94.0)
- moved R2 17.7 mm to (132.9, 87.8), turned to 90 degrees
- moved R3 14.6 mm to (136.6, 91.2)
- moved R1 10.3 mm to (143.2, 87.8), turned to 90 degrees
- moved U2 8.38 mm to (141.1, 97.1), turned to 90 degrees
- moved U1 7.14 mm to (135.0, 97.1), turned to 90 degrees
- moved J1 0.20 mm to (138.1, 86.0)
Routing:
- net /SCL: track 0.00 -> 27.1 mm
- net /TMP_ALERT: track 0.00 -> 19.7 mm
- net /SDA: track 0.00 -> 17.6 mm
- net /VCC: track 0.00 -> 14.1 mm, vias 0 -> 1
- net /GND: track 0.00 -> 3.98 mm, vias 0 -> 1
Other:
- board outline added: 12.9 x 17.5 mm
- rule pad_to_mask_clearance: 0 -> 0.05

Commit message: csv document
Routing:
- net /VCC: track 14.1 -> 13.6 mm, vias 1 -> 2
- net (no net): vias 0 -> 2
Changed lines of the file:
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@@
   (gr_line (start 131.6 99.24) (end 131.599858 82.449999)
     (stroke (width 0.1) (type default)) (layer "Edge.Cuts"))
+  (via (at 138.88 94.9) (size 0.5) (drill 0.25) (layers "F.Cu" "B.Cu") (net 0))
+  (via (at 137.31 96.93) (size 0.5) (drill 0.25) (layers "F.Cu" "B.Cu") (net 0))
   (segment (start 135.5385 89.8315) (end 135.5385 89.8485) (width 0.7) (layer "F.Cu") (net 1))
   (segment (start 135.64 92.57) (end 135.6375 92.5725) (width 0.7) (layer "F.Cu") (net 1))
@@
   (segment (start 140.2375 94) (end 140.2375 91.65) (width 1) (layer "F.Cu") (net 1))
   (segment (start 135.5385 87.950001) (end 135.5385 89.8285) (width 0.7) (layer "F.Cu") (net 1))
-  (segment (start 135.399999 96.3531) (end 136.6869 96.3531) (width 0.3) (layer "F.Cu") (net 1))
   (segment (start 135.6375 93.775) (end 135.8625 94) (width 0.7) (layer "F.Cu") (net 1))
   (segment (start 135.54 89.83) (end 135.5385 89.8315) (width 0.7) (layer "F.Cu") (net 1))
@@
   (segment (start 140.2375 91.65) (end 143.225 88.6625) (width 1) (layer "F.Cu") (net 1))
   (segment (start 135.5385 89.8285) (end 135.54 89.83) (width 0.7) (layer "F.Cu") (net 1))
+  (segment (start 135.399999 96.3531) (end 136.2631 96.3531) (width 0.3) (layer "F.Cu") (net 1))
   (segment (start 135.5385 91.051) (end 135.6375 91.15) (width 0.7) (layer "F.Cu") (net 1))
+  (via (at 136.43 96.93) (size 0.5) (drill 0.25) (layers "F.Cu" "B.Cu") (net 1))
   (via (at 135.54 89.85) (size 0.7) (drill 0.4) (layers "F.Cu" "B.Cu") (net 1))
   (segment (start 141.9625 92.7725) (end 141.96 92.77) (width 1) (layer "F.Cu") (net 2))
